Commit message: Updated model of the robot along with lidar added to it

File: task1/urdf/bot_desc.urdf (robot description, URDF)
Before this commit: robot diff_drive, 4 links, 3 joints
Links:
- added link base_footprint
- added link caster_wheel, mass 0.5; collision mesh filename=file:///home/sanjit/ros2_ws/src/task1/mesh/caster_wheel.STL; visual mesh filename=file:///home/sanjit/ros2_ws/src/task1/mesh/caster_wheel.STL
- added link lidar_cylinder, mass 0.1; collision cylinder length=0.05 radius=0.06; visual cylinder length=0.05 radius=0.06
- link base_link: mass None -> 3.0; geometry collision mesh filename=file:///home/sanjit/ros2_ws/src/task1/mesh/bot_body.stl; visual mesh filename=file:///home/sanjit/ros2_ws/src/task1/mesh/bot_body.stl
- link caster_part: mass None -> 0.5; geometry collision mesh filename=file:///home/sanjit/ros2_ws/src/task1/mesh/caster_part.STL; visual mesh filename=file:///home/sanjit/ros2_ws/src/task1/mesh/caster_part.STL
- link left_wheel: mass None -> 0.5; geometry collision mesh filename=file:///home/sanjit/ros2_ws/src/task1/mesh/wheel.STL; visual mesh filename=file:///home/sanjit/ros2_ws/src/task1/mesh/wheel.STL
- link right_wheel: mass None -> 0.5; geometry collision mesh filename=file:///home/sanjit/ros2_ws/src/task1/mesh/wheel.STL; visual mesh filename=file:///home/sanjit/ros2_ws/src/task1/mesh/wheel.STL
Joints:
- removed joint caster_part_joint
- added joint base_joint: type fixed, parent base_footprint, child base_link, origin xyz=0.0 0.0 0.1 rpy=0.0 0.0 0.0
- added joint caster_wheel_joint: type continuous, parent caster_part, child caster_wheel, origin xyz=0.0 0.15 0.0 rpy=0.0 0.0 0.0, axis 1.0 0.0 0.0
- added joint lidar_joint: type fixed, parent base_link, child lidar_cylinder, origin xyz=0.0 0 2.0 rpy=0.0 0.0 0.0, axis 0.0 0.0 0.0
- added joint part_joint: type continuous, parent base_link, child caster_part, origin xyz=0.0 1.0 0.0 rpy=-1.57 0.0 0.0, axis 0.0 1.0 0.0
- joint left_wheel_joint: axis (none) -> 1.0 0.0 0.0; origin xyz=-1.0 -1.6 0.4 rpy=0.0 0.0 0.0 -> xyz=-1.2 -1.0 0.1 rpy=0.0 0.0 0.0
- joint right_wheel_joint: axis (none) -> 1.0 0.0 0.0; origin xyz=1.19 -1.6 0.4 rpy=0.0 0.0 0.0 -> xyz=1.2 -1.0 0.1 rpy=0.0 0.0 0.0
