Commit message: scaled down the bot

File: install/task1/share/task1/urdf/bot_desc.urdf (robot description, URDF)
Before this commit: robot diff_drive, 7 links, 6 joints
Links:
- link base_link: geometry collision mesh filename=file:///home/sanjit/ros2_ws/src/task1/mesh/bot_body.stl; visual mesh filename=file:///home/sanjit/ros2_ws/src/task1/mesh/bot_body.stl
- link caster_part: geometry collision mesh filename=file:///home/sanjit/ros2_ws/src/task1/mesh/caster_part.STL; visual mesh filename=file:///home/sanjit/ros2_ws/src/task1/mesh/caster_part.STL
- link caster_wheel: geometry collision mesh filename=file:///home/sanjit/ros2_ws/src/task1/mesh/caster_wheel.STL; visual mesh filename=file:///home/sanjit/ros2_ws/src/task1/mesh/caster_wheel.STL
Joints:
- joint base_joint: origin xyz=0.5 0.5 0.0 rpy=0.0 0.0 0.0 -> xyz=0.0 0.0 0.1 rpy=0.0 0.0 0.0
- joint caster_wheel_joint: origin xyz=0.0 0.045 0.02 rpy=0.0 0.0 0.0 -> xyz=0.0 0.15 0.0 rpy=0.0 0.0 0.0
- joint left_wheel_joint: axis -1.0 0.0 0.0 -> 1.0 0.0 0.0; origin xyz=-0.4 -0.36 0.14 rpy=0.0 0.0 0.0 -> xyz=-1.2 -1.0 0.1 rpy=0.0 0.0 0.0
- joint lidar_joint: origin xyz=0.0 0 0.5 rpy=0.0 0.0 0.0 -> xyz=0.0 0 2.0 rpy=0.0 0.0 0.0
- joint part_joint: origin xyz=0.0 0.25 0.0 rpy=-1.57 0.0 0.0 -> xyz=0.0 1.0 0.0 rpy=-1.57 0.0 0.0
- joint right_wheel_joint: axis -1.0 0.0 0.0 -> 1.0 0.0 0.0; origin xyz=0.4 -0.36 0.14 rpy=0.0 0.0 0.0 -> xyz=1.2 -1.0 0.1 rpy=0.0 0.0 0.0

Commit message: tested movement in two coordinates

File: install/task1/share/task1/urdf/bot_desc.urdf (robot description, URDF)
Before this commit: robot diff_drive, 7 links, 6 joints
Links:
- link base_link: geometry collision mesh filename=file:///home/sanjit/ros2_ws/src/task1/mesh/bot_body.stl scale=0.25 0.25 0.25; visual mesh filename=file:///home/sanjit/ros2_ws/src/task1/mesh/bot_body.stl scale=0.25 0.25 0.25
- link caster_part: geometry collision mesh filename=file:///home/sanjit/ros2_ws/src/task1/mesh/caster_part.STL scale=0.3 0.3 0.3; visual mesh filename=file:///home/sanjit/ros2_ws/src/task1/mesh/caster_part.STL scale=0.3 0.3 0.3
- link caster_wheel: geometry collision mesh filename=file:///home/sanjit/ros2_ws/src/task1/mesh/caster_wheel.STL scale=0.3 0.3 0.3; visual mesh filename=file:///home/sanjit/ros2_ws/src/task1/mesh/caster_wheel.STL scale=0.3 0.3 0.3
Joints:
- joint base_joint: origin xyz=0.0 0.0 0.1 rpy=0.0 0.0 0.0 -> xyz=0.0 0.0 0.0 rpy=0.0 0.0 0.0
- joint caster_wheel_joint: origin xyz=0.0 0.15 0.0 rpy=0.0 0.0 0.0 -> xyz=0.0 0.045 0.02 rpy=0.0 0.0 0.0
- joint left_wheel_joint: axis 1.0 0.0 0.0 -> -1.0 0.0 0.0; origin xyz=-1.2 -1.0 0.1 rpy=0.0 0.0 0.0 -> xyz=-0.4 -0.36 0.14 rpy=0.0 0.0 0.0
- joint lidar_joint: origin xyz=0.0 0 2.0 rpy=0.0 0.0 0.0 -> xyz=0.0 0 0.5 rpy=0.0 0.0 0.0
- joint part_joint: origin xyz=0.0 1.0 0.0 rpy=-1.57 0.0 0.0 -> xyz=0.0 0.25 0.0 rpy=-1.57 0.0 0.0
- joint right_wheel_joint: axis 1.0 0.0 0.0 -> -1.0 0.0 0.0; origin xyz=1.2 -1.0 0.1 rpy=0.0 0.0 0.0 -> xyz=0.4 -0.36 0.14 rpy=0.0 0.0 0.0

File: task1/urdf/bot_desc.urdf (robot description, URDF)
Before this commit: robot diff_drive, 7 links, 6 joints
Links:
- link base_link: geometry collision mesh filename=file:///home/sanjit/ros2_ws/src/task1/mesh/bot_body.stl scale=0.18 0.18 0.18; visual mesh filename=file:///home/sanjit/ros2_ws/src/task1/mesh/bot_body.stl scale=0.20 0.20 0.20
- link caster_part: geometry visual mesh filename=file:///home/sanjit/ros2_ws/src/task1/mesh/caster_part.STL scale=0.3 0.3 0.3
Joints:
- joint left_wheel_joint: origin xyz=-0.4 -0.36 0.14 rpy=0.0 0.0 0.0 -> xyz=-0.30 -0.36 0.14 rpy=0.0 0.0 0.0
- joint part_joint: origin xyz=0.0 0.25 0.0 rpy=-1.57 0.0 0.0 -> xyz=0.0 0.20 0.05 rpy=-1.57 0.0 0.0
- joint right_wheel_joint: origin xyz=0.4 -0.36 0.14 rpy=0.0 0.0 0.0 -> xyz=0.3 -0.36 0.14 rpy=0.0 0.0 0.0
